Commit message: integrated a public aruco repo

File: src/grap_description/urdf/real_camera.urdf.xacro (robot description, xacro)
@@ -74,5 +74,5 @@
     <!-- camera color joints and links -->
     <joint name="camera_color_joint" type="fixed">
-        <origin xyz="0 0.015 0" rpy="0 0 0" />
+        <origin xyz="0 0.015 0" rpy="0 0 ${-M_PI/2}" />
         <parent link="camera_link" />
         <child link="camera_color_frame" />

Commit message: yolo detection depth move program

File: src/grap_description/urdf/real_camera.urdf.xacro (robot description, xacro)
@@ -55,5 +55,5 @@
     </link>
   <joint name="camera_joint" type="fixed">
-    <origin xyz="0 0 0.1" rpy="0 0 ${M_PI/2}"/>
+    <origin xyz="0 0.05 0.05" rpy="0 0 ${M_PI/2}"/>
     <parent link="gripper"/>
     <child link="camera_link"/>
